Commit message: autobotware benchmarking world, edits in the robot model, and SGM clustering algorithm.

File: autobotware_simulator/urdf/velodyne/skid_steer_bot.xacro (robot description, xacro)
@@ -329,5 +329,5 @@
   <joint type="fixed" name="coloredLidar_joint">
     <!--<origin xyz="${laser_x_offset} 0 ${laser_z_offset}" rpy="0 0 0"/>-->
-    <origin xyz="0.2 0 0.3" rpy="0 0 0"/>
+    <origin xyz="0.2 0 1.5" rpy="0 0 0"/>
     <child link="coloredLidar"/>
     <parent link="chassis"/>

Commit message: fixing the hight of the velodyne sensor

File: autobotware_simulator/urdf/velodyne/skid_steer_bot.xacro (robot description, xacro)
@@ -329,5 +329,5 @@
   <joint type="fixed" name="coloredLidar_joint">
     <!--<origin xyz="${laser_x_offset} 0 ${laser_z_offset}" rpy="0 0 0"/>-->
-    <origin xyz="0.2 0 1.5" rpy="0 0 0"/>
+    <origin xyz="0.2 0 0.5" rpy="0 0 0"/>
     <child link="coloredLidar"/>
     <parent link="chassis"/>
