Commit message: changing framework name from autobotware to modulidar

File: gazebo_simulator/urdf/benwake/skid_steer_bot.xacro (robot description, xacro)
@@ -1,5 +1,5 @@
 <?xml version='1.0'?>
 <robot name="skid_steer_bot" xmlns:xacro="http://www.ros.org/wiki/xacro">
-  <xacro:include filename="$(find autobotware_simulator)/urdf/benwake/skid_steer_bot.gazebo" />
+  <xacro:include filename="$(find gazebo_simulator)/urdf/benwake/skid_steer_bot.gazebo" />
   <!-- Scale the robot size to fit the environment -->
   <xacro:property name="scale" value="1.0" />
@@ -323,5 +323,5 @@
       <origin xyz="0 0 0" rpy=" 0 0 0"/>
       <geometry>
-        <mesh filename="package://autobotware_simulator/meshes/hokuyo.dae"/>
+        <mesh filename="package://gazebo_simulator/meshes/hokuyo.dae"/>
       </geometry>
     </visual>
@@ -357,5 +357,5 @@
       <origin xyz="0 0 0" rpy=" 0 0 0"/>
       <geometry>
-        <mesh filename="package://autobotware_simulator/meshes/hokuyo.dae"/>
+        <mesh filename="package://gazebo_simulator/meshes/hokuyo.dae"/>
       </geometry>
     </visual>

File: gazebo_simulator/urdf/velodyne/skid_steer_bot.xacro (robot description, xacro)
@@ -1,5 +1,5 @@
 <?xml version='1.0'?>
 <robot name="skid_steer_bot" xmlns:xacro="http://www.ros.org/wiki/xacro">
-  <xacro:include filename="$(find autobotware_simulator)/urdf/velodyne/skid_steer_bot.gazebo" />
+  <xacro:include filename="$(find gazebo_simulator)/urdf/velodyne/skid_steer_bot.gazebo" />
   <!-- Scale the robot size to fit the environment -->
   <xacro:property name="scale" value="1.0" />
@@ -323,5 +323,5 @@
       <origin xyz="0 0 0" rpy=" 0 0 0"/>
       <geometry>
-        <mesh filename="package://autobotware_simulator/meshes/hokuyo.dae"/>
+        <mesh filename="package://gazebo_simulator/meshes/hokuyo.dae"/>
       </geometry>
     </visual>
